Commit message: update urdf

File: resources/robots/go2/urdf/go2.urdf (robot description, URDF)
Before this commit: robot go2_description, 33 links, 32 joints
Joints:
- joint FL_calf_joint: limit lower=-2.7227 upper=-0.83776 effort=35.55 velocity=20.07 -> lower=-2.7227 upper=-0.83776 effort=45.43 velocity=15.70
- joint FR_calf_joint: limit lower=-2.7227 upper=-0.83776 effort=35.55 velocity=20.07 -> lower=-2.7227 upper=-0.83776 effort=45.43 velocity=15.70
- joint RL_calf_joint: limit lower=-2.7227 upper=-0.83776 effort=35.55 velocity=20.07 -> lower=-2.7227 upper=-0.83776 effort=45.43 velocity=15.70
- joint RR_calf_joint: limit lower=-2.7227 upper=-0.83776 effort=35.55 velocity=20.07 -> lower=-2.7227 upper=-0.83776 effort=45.43 velocity=15.70
- joint back_dorsal_joint: limit lower=-0.5 upper=0.5 effort=60 velocity=20.73 -> (none); type revolute -> fixed
- joint front_dorsal_joint: limit lower=-1 upper=1 effort=60 velocity=20.73 -> (none); type revolute -> fixed

Commit message: before big change

File: resources/robots/go2/urdf/go2.urdf (robot description, URDF)
Before this commit: robot go2_description, 33 links, 32 joints
Joints:
- joint FL_hip_joint: limit lower=-1.0472 upper=1.0472 effort=23.7 velocity=30.1 -> lower=-1.0472 upper=1.0472 effort=33.7 velocity=30.1
- joint FL_thigh_joint: limit lower=-1.5708 upper=3.4907 effort=23.7 velocity=30.1 -> lower=-1.5708 upper=3.4907 effort=33.7 velocity=30.1
- joint FR_hip_joint: limit lower=-1.0472 upper=1.0472 effort=23.7 velocity=30.1 -> lower=-1.0472 upper=1.0472 effort=33.7 velocity=30.1
- joint FR_thigh_joint: limit lower=-1.5708 upper=3.4907 effort=23.7 velocity=30.1 -> lower=-1.5708 upper=3.4907 effort=33.7 velocity=30.1
- joint RL_hip_joint: limit lower=-1.0472 upper=1.0472 effort=23.7 velocity=30.1 -> lower=-1.0472 upper=1.0472 effort=33.7 velocity=30.1
- joint RL_thigh_joint: limit lower=-0.5236 upper=4.5379 effort=23.7 velocity=30.1 -> lower=-0.5236 upper=4.5379 effort=33.7 velocity=30.1
- joint RR_hip_joint: limit lower=-1.0472 upper=1.0472 effort=23.7 velocity=30.1 -> lower=-1.0472 upper=1.0472 effort=33.7 velocity=30.1
- joint RR_thigh_joint: limit lower=-0.5236 upper=4.5379 effort=23.7 velocity=30.1 -> lower=-0.5236 upper=4.5379 effort=33.7 velocity=30.1

Commit message: 12.17

File: resources/robots/go2/urdf/go2.urdf (robot description, URDF)
Before this commit: robot go2_description, 33 links, 32 joints
Joints:
- joint FL_hip_joint: limit lower=-1.0472 upper=1.0472 effort=33.7 velocity=30.1 -> lower=-1.0472 upper=1.0472 effort=23.7 velocity=30.1
- joint FL_thigh_joint: limit lower=-1.5708 upper=3.4907 effort=33.7 velocity=30.1 -> lower=-1.5708 upper=3.4907 effort=23.7 velocity=30.1
- joint FR_hip_joint: limit lower=-1.0472 upper=1.0472 effort=33.7 velocity=30.1 -> lower=-1.0472 upper=1.0472 effort=23.7 velocity=30.1
- joint FR_thigh_joint: limit lower=-1.5708 upper=3.4907 effort=33.7 velocity=30.1 -> lower=-1.5708 upper=3.4907 effort=23.7 velocity=30.1
- joint RL_hip_joint: limit lower=-1.0472 upper=1.0472 effort=33.7 velocity=30.1 -> lower=-1.0472 upper=1.0472 effort=23.7 velocity=30.1
- joint RL_thigh_joint: limit lower=-0.5236 upper=4.5379 effort=33.7 velocity=30.1 -> lower=-0.5236 upper=4.5379 effort=23.7 velocity=30.1
- joint RR_hip_joint: limit lower=-1.0472 upper=1.0472 effort=33.7 velocity=30.1 -> lower=-1.0472 upper=1.0472 effort=23.7 velocity=30.1
- joint RR_thigh_joint: limit lower=-0.5236 upper=4.5379 effort=33.7 velocity=30.1 -> lower=-0.5236 upper=4.5379 effort=23.7 velocity=30.1
- joint back_dorsal_joint: limit (none) -> lower=-0.5 upper=0.5 effort=60 velocity=20.73; type fixed -> revolute
- joint front_dorsal_joint: limit (none) -> lower=-1 upper=1 effort=60 velocity=20.73; type fixed -> revolute

Commit message: update final

File: resources/robots/go2/urdf/go2.urdf (robot description, URDF)
Before this commit: robot go2_description, 33 links, 32 joints
Links:
- link back_body: mass 0 -> 0.92
